File: es 3/es 3.sch (KiCad schematic (older format))
At the start: 11 parts, among them P1 Power, P2 Analog, P3 Digital, P4 Digital, P5 CONN_01X01, P6 CONN_01X01, P7 CONN_01X01, P8 CONN_01X01

Commit message: DHT11+Termocoppia
Parts:
- added U?: DHT11, symbol Sensor:DHT11
- IC?: symbol MAX6675ISA:MAX6675ISA -> es-3-rescue:MAX6675ISA-MAX6675ISA
Connections:
- wire segments 73 -> 78
Other:
- note removed: "Shield for Arduino that uses\nthe same pin disposition\nlike "Uno" board Rev 3."
- moved on the sheet: IC?, J?, P1, P2, P3, P4, P5, P6, P7, P8, TC?
